File: LM358-5-12V-amp.kicad_pcb (KiCad board)
At the start: 2 copper layers, 76.2 x 57.1 mm, 30 parts, among them J1 IN1, J2 IN2, J3 Barrel_Jack, M1 Fan_3pin, M2 Fan_3pin, Q1 PN2222A, Q2 PN2222A, U1 WeMos_D1_mini, U2 L7805, U3 LM358

Commit message: added trim pots and TO220 transistor
Parts:
- added RV1: 5k, Potentiometer_THT:Potentiometer_Bourns_3296W_Vertical, F.Cu at (214.6, 25.4)
- added RV2: 5k, Potentiometer_THT:Potentiometer_Bourns_3296W_Vertical, F.Cu at (119.4, 157.5)
- added RV3: 5k, Potentiometer_THT:Potentiometer_Bourns_3296W_Vertical, F.Cu at (170.2, 91.4)
- added RV4: 5k, Potentiometer_THT:Potentiometer_Bourns_3296W_Vertical, F.Cu at (198.1, 24.1)
- J2: value IN2 -> IN1
- Q1, Q2: value PN2222A -> TIP120; footprint Package_TO_SOT_THT:TO-92_Inline -> Package_TO_SOT_THT:TO-220-3_Vertical
- R3, R5: value 6.8k -> 3k
- R7, R8: value 2.2k -> 1.5k
- moved C2 168.2 mm to (265.4, 141.0), turned to 0 degrees
- moved J1 162.8 mm to (248.4, 143.7), turned to 0 degrees
- moved R11 148.5 mm to (249.0, 81.2), turned to 0 degrees
- moved M1 146.1 mm to (241.3, 54.6), turned to 0 degrees
- moved R4 125.2 mm to (224.8, 35.6), turned to 0 degrees
- moved R7 121.1 mm to (237.3, 128.5)
- moved R2 121.0 mm to (59.4, 125.1)
- moved C1 120.9 mm to (260.4, 109.2), turned to 0 degrees
- moved C3 120.0 mm to (265.4, 154.9), turned to 0 degrees
- moved J2 115.7 mm to (270.5, 123.2), turned to 0 degrees
- moved C4 114.4 mm to (259.1, 132.1)
- moved D1 107.1 mm to (197.5, 38.8)
- moved R13 102.2 mm to (194.3, 154.9), turned to 0 degrees
- moved M2 101.9 mm to (256.5, 54.6), turned to 0 degrees
- moved U1 101.4 mm to (31.3, 32.8)
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Connections:
- Q1 pad 1: Net-(D1-Pad2) -> Net-(Q1-Pad1)
- Q1 pad 2: Net-(Q1-Pad2) -> 14VDC
- Q1 pad 3: 14VDC -> Net-(D1-Pad2)
- Q2 pad 1: Net-(D2-Pad2) -> Net-(Q2-Pad1)
- Q2 pad 2: Net-(Q2-Pad2) -> 14VDC
- Q2 pad 3: 14VDC -> Net-(D2-Pad2)
- R10 pad 1: Net-(Q2-Pad2) -> Net-(Q2-Pad1)
- R5 pad 1: Net-(R10-Pad2) -> Net-(R5-Pad1)
- R7 pad 1: GND -> Net-(R7-Pad1)
- R7 pad 2: Net-(R4-Pad1) -> GND
- R8 pad 1: GND -> Net-(R8-Pad1)
- R8 pad 2: Net-(R6-Pad1) -> GND
- R9 pad 1: Net-(Q1-Pad2) -> Net-(Q1-Pad1)
- R9 pad 2: Net-(R3-Pad1) -> Net-(R9-Pad2)
- U1 pad 1: 5VDC -> (no net)
- U1 pad 13: Net-(U1-Pad13) -> (no net)
- U1 pad 14: Net-(U1-Pad14) -> (no net)
- U1 pad 15: Net-(U1-Pad15) -> (no net)
- U1 pad 16: Net-(U1-Pad16) -> (no net)
- U1 pad 4: Net-(U1-Pad4) -> (no net)
- U1 pad 5: Net-(U1-Pad5) -> (no net)
- U1 pad 6: Net-(U1-Pad6) -> (no net)
- U1 pad 7: Net-(U1-Pad7) -> (no net)
- U1 pad 8: Net-(U1-Pad8) -> (no net)
- U3 pad 1: Net-(Q1-Pad2) -> Net-(Q1-Pad1)
- U3 pad 2: Net-(R3-Pad1) -> Net-(RV3-Pad2)
- U3 pad 3: Net-(R4-Pad1) -> Net-(RV1-Pad2)
- U3 pad 5: Net-(R6-Pad1) -> Net-(RV2-Pad2)
- U3 pad 6: Net-(R10-Pad2) -> Net-(RV4-Pad2)
- U3 pad 7: Net-(Q2-Pad2) -> Net-(Q2-Pad1)
Routing:
- net 14VDC: track 155.3 -> 0.00 mm
- net 5VDC: track 105.3 -> 0.00 mm
- net TACH2: track 67.5 -> 0.00 mm
- net Net-(Q2-Pad2): track 60.4 -> 0.00 mm
- net PWM1: track 52.3 -> 0.00 mm
- net TACH1: track 49.3 -> 0.00 mm
- net Net-(Q1-Pad2): track 48.2 -> 0.00 mm
- net Net-(C3-Pad1): track 46.5 -> 0.00 mm
- net Net-(C2-Pad1): track 42.1 -> 0.00 mm
- net PWM2: track 40.3 -> 0.00 mm
- net Net-(D2-Pad2): track 31.6 -> 0.00 mm
- net Net-(D1-Pad2): track 30.3 -> 0.00 mm
- net Net-(R10-Pad2): track 21.8 -> 0.00 mm
- net Net-(R3-Pad1): track 20.7 -> 0.00 mm
- net Net-(R4-Pad1): track 15.0 -> 0.00 mm
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- removed copper zone on B.Cu, net GND
- removed copper zone on F.Cu, net GND
Other:
- board outline removed
- board text removed: "+"
