File: LM358-5-12V-amp.sch (KiCad schematic (older format))
At the start: 30 parts, among them J1 IN1, J2 IN2, J3 Barrel_Jack, M1 Fan_3pin, M2 Fan_3pin, Q1 PN2222A, Q2 PN2222A, U1 WeMos_D1_mini, U2 L7805, U3 LM358

Commit message: added trim pots and TO220 transistor
Parts:
- removed Q2: PN2222A, Package_TO_SOT_THT:TO-92_Inline, symbol Transistor_BJT:PN2222A
- added Q2: TIP120, Package_TO_SOT_THT:TO-220-3_Vertical, symbol Transistor_BJT:TIP120
- added RV1, RV2, RV3, RV4: 5k, Potentiometer_THT:Potentiometer_Bourns_3296W_Vertical, symbol Device:R_POT_TRIM_US
- J2: value IN2 -> IN1
- Q1: value PN2222A -> TIP120; footprint Package_TO_SOT_THT:TO-92_Inline -> Package_TO_SOT_THT:TO-220-3_Vertical; symbol Transistor_BJT:PN2222A -> Transistor_BJT:TIP120
- R10: value 15k -> 20k
Connections:
- wire segments 96 -> 100
- no-connect marks 8 -> 9
Other:
- moved on the sheet: C2, D1, J1, M1, R1, R11, R13, R3, R4, R7, R9, U1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

Commit message: different voltage?
Parts:
- RV1, RV2, RV3, RV4: value 5k -> 500
Changed lines of the file:
@@
 P 5200 2950
 F 0 "RV3" H 5132 2996 50  0000 R CNN
-F 1 "5k" H 5150 3100 50  0000 R CNN
+F 1 "500" H 5150 3100 50  0000 R CNN
 F 2 "Potentiometer_THT:Potentiometer_Bourns_3296W_Vertical" H 5200 2950 50  0001 C CNN
 F 3 "~" H 5200 2950 50  0001 C CNN
@@
 P 5100 3450
 F 0 "RV1" H 5050 3500 50  0000 R CNN
-F 1 "5k" H 5000 3600 50  0000 R CNN
+F 1 "500" H 5000 3600 50  0000 R CNN
 F 2 "Potentiometer_THT:Potentiometer_Bourns_3296W_Vertical" H 5100 3450 50  0001 C CNN
 F 3 "~" H 5100 3450 50  0001 C CNN
@@
 P 5200 4900
 F 0 "RV4" H 5132 4946 50  0000 R CNN
-F 1 "5k" H 5150 5050 50  0000 R CNN
+F 1 "500" H 5150 5050 50  0000 R CNN
 F 2 "Potentiometer_THT:Potentiometer_Bourns_3296W_Vertical" H 5200 4900 50  0001 C CNN
 F 3 "~" H 5200 4900 50  0001 C CNN
@@
 P 5100 5400
 F 0 "RV2" H 5050 5450 50  0000 R CNN
-F 1 "5k" H 5000 5550 50  0000 R CNN
+F 1 "500" H 5000 5550 50  0000 R CNN
 F 2 "Potentiometer_THT:Potentiometer_Bourns_3296W_Vertical" H 5100 5400 50  0001 C CNN
 F 3 "~" H 5100 5400 50  0001 C CNN
