File: randall-LM358-5-12V-amp.sch (KiCad schematic (older format))
At the start: 27 parts, among them J1 Barrel_Jack, M1 Fan_3pin, M2 Fan_3pin, Q1 TIP120, Q2 TIP120, U1 LM2674M-3.3, U2 LM358, U3 Z-Uno-Module

Commit message: Ok this is probably wrong due to Via use?
Parts:
- added J2: AVR-ISP-6, Connector_PinHeader_2.54mm:PinHeader_2x03_P2.54mm_Vertical, symbol Connector:AVR-ISP-6
Connections:
- net +3V3: now also J2.2 (VCC)
- net GND: now also J2.6 (GND)
- net SCK: now reaches U3.0 (SCK)
- net SCK: now also J2.3 (SCK)
- net MISO: now reaches U3.1 (MISO)
- net MISO: now also J2.1 (MISO)
- net MOSI: now reaches U3.2 (MOSI)
- net MOSI: now also J2.4 (MOSI)
- net RST: now reaches U3.30 (RST_N)
- net RST: now also J2.5 (~RST)
- no-connect marks 27 -> 44
Changed lines of the file:
@@
 	1    0    0    -1
 $EndComp
-NoConn ~ 1900 2750
 NoConn ~ 1800 2750
 NoConn ~ 1700 2750
-NoConn ~ 1100 3250
-NoConn ~ 1100 3350
-NoConn ~ 1100 3450
 NoConn ~ 1100 3650
 NoConn ~ 1100 3750
@@
 NoConn ~ 3000 3550
 NoConn ~ 3000 3650
+NoConn ~ 1300 3650
+NoConn ~ 1300 3750
+NoConn ~ 1300 3950
+NoConn ~ 1300 4050
+NoConn ~ 1300 4150
+NoConn ~ 1300 4250
+NoConn ~ 1300 4450
+NoConn ~ 1300 4550
+NoConn ~ 2800 4950
+NoConn ~ 2800 4850
+NoConn ~ 2800 4750
+NoConn ~ 2800 4650
+NoConn ~ 2800 3650
+NoConn ~ 2800 3550
+NoConn ~ 2800 3450
+NoConn ~ 2800 3350
+NoConn ~ 2800 3250
+NoConn ~ 1800 2950
+NoConn ~ 1700 2950
+NoConn ~ 3400 3800
+NoConn ~ 3750 4150
+$Comp
+L Connector:AVR-ISP-6 J2
+U 1 1 608E7125
+P 2150 6300
+F 0 "J2" H 1820 6304 50  0000 R CNN
+F 1 "AVR-ISP-6" H 1820 6395 50  0000 R CNN
+F 2 "Connector_PinHeader_2.54mm:PinHeader_2x03_P2.54mm_Vertical" V 1900 6350 50  0001 C CNN
+F 3 " ~" H 875 5750 50  0001 C CNN
+	1    2150 6300
+	-1   0    0    1
+$EndComp
+Text GLabel 1100 3250 0    50   Input ~ 0
+SCK
+Text GLabel 1750 6300 0    50   Output ~ 0
+SCK
+Text GLabel 1100 3350 0    50   Input ~ 0
+MISO
+Text GLabel 1100 3450 0    50   Input ~ 0
+MOSI
+Text GLabel 1750 6500 0    50   Output ~ 0
+MISO
+Text GLabel 1750 6400 0    50   Output ~ 0
+MOSI
+Text GLabel 1900 2750 1    50   Input ~ 0
+RST
+$Comp
+L power:GND #PWR020
+U 1 1 608FEC8A
+P 2250 5900
+F 0 "#PWR020" H 2250 5650 50  0001 C CNN
+F 1 "GND" H 2255 5727 50  0000 C CNN
+F 2 "" H 2250 5900 50  0001 C CNN
+F 3 "" H 2250 5900 50  0001 C CNN
+	1    2250 5900
+	-1   0    0    1
+$EndComp
+Text GLabel 1750 6200 0    50   Output ~ 0
+RST
+Text GLabel 2250 6800 3    50   Output ~ 0
+3V3DC
 $EndSCHEMATC
