File: randall-LM358-5-12V-amp.sch (KiCad schematic (older format))
At the start: 25 parts, among them J1 IN1, J3 Barrel_Jack, M1 Fan_3pin, M2 Fan_3pin, Q1 TIP120, Q2 TIP120, U1 xl6009_buckboost, U2 MP1584EN, U3 LM358, U4 Z-Uno

Commit message: Update gitignore
Parts:
- gave numbers to parts that had none: 2
Connections:
- wire segments 83 -> 84
Changed lines of the file:
@@
 	1    0    0    -1
 $EndComp
-Text GLabel 7800 1600 2    50   Input ~ 0
-10-24VDC+
-Text GLabel 7800 1800 2    50   Input ~ 0
-10-24VDC-
 Wire Wire Line
 	7800 1800 7750 1800
 Wire Wire Line
 	7750 1600 7800 1600
-$Comp
-L power:GND #PWR07
-U 1 1 60517F01
-P 3400 1850
-F 0 "#PWR07" H 3400 1600 50  0001 C CNN
-F 1 "GND" H 3405 1677 50  0000 C CNN
-F 2 "" H 3400 1850 50  0001 C CNN
-F 3 "" H 3400 1850 50  0001 C CNN
-	1    3400 1850
-	1    0    0    -1
-$EndComp
 Text GLabel 2550 3650 2    50   Input ~ 0
 PWM1
@@
 	5450 2650 5700 2650
 $Comp
-L power:GND #PWR?
+L power:GND #PWR0101
 U 1 1 607AF4E1
 P 4350 2500
-F 0 "#PWR?" H 4350 2250 50  0001 C CNN
+F 0 "#PWR0101" H 4350 2250 50  0001 C CNN
 F 1 "GND" H 4355 2327 50  0000 C CNN
 F 2 "" H 4350 2500 50  0001 C CNN
@@
 	7550 6050 7550 6000
 $Comp
-L Connector:Conn_01x02_Male J?
+L Connector:Conn_01x02_Male J2
 U 1 1 607E39A3
 P 3600 5350
-F 0 "J?" H 3550 5300 50  0000 C CNN
+F 0 "J2" H 3550 5300 50  0000 C CNN
 F 1 "IN2" H 3450 5400 50  0000 C CNN
 F 2 "Connector_PinHeader_2.54mm:PinHeader_1x02_P2.54mm_Vertical" H 3600 5350 50  0001 C CNN
@@
 	7150 4950 6650 4950
 $Comp
-L power:VCC #PWR?
+L power:VCC #PWR0102
 U 1 1 607E39B9
 P 6650 4900
-F 0 "#PWR?" H 6650 4750 50  0001 C CNN
+F 0 "#PWR0102" H 6650 4750 50  0001 C CNN
 F 1 "VCC" H 6665 5073 50  0000 C CNN
 F 2 "" H 6650 4900 50  0001 C CNN
@@
 Connection ~ 6650 4950
 $Comp
-L power:GND #PWR?
+L power:GND #PWR0103
 U 1 1 607E39C1
 P 3800 5600
-F 0 "#PWR?" H 3800 5350 50  0001 C CNN
+F 0 "#PWR0103" H 3800 5350 50  0001 C CNN
 F 1 "GND" H 3805 5427 50  0000 C CNN
 F 2 "" H 3800 5600 50  0001 C CNN
@@
 $EndComp
 $Comp
-L power:GND #PWR?
+L power:GND #PWR0104
 U 1 1 607E39C7
 P 4550 5900
-F 0 "#PWR?" H 4550 5650 50  0001 C CNN
+F 0 "#PWR0104" H 4550 5650 50  0001 C CNN
 F 1 "GND" H 4555 5727 50  0000 C CNN
 F 2 "" H 4550 5900 50  0001 C CNN
@@
 	4550 5800 4550 5900
 $Comp
-L power:GND #PWR?
+L power:GND #PWR0105
 U 1 1 607E39CE
 P 6650 5850
-F 0 "#PWR?" H 6650 5600 50  0001 C CNN
+F 0 "#PWR0105" H 6650 5600 50  0001 C CNN
 F 1 "GND" H 6655 5677 50  0000 C CNN
 F 2 "" H 6650 5850 50  0001 C CNN
@@
 $EndComp
 $Comp
-L power:GND #PWR?
+L power:GND #PWR0106
 U 1 1 607E39D4
 P 7550 6050
-F 0 "#PWR?" H 7550 5800 50  0001 C CNN
+F 0 "#PWR0106" H 7550 5800 50  0001 C CNN
 F 1 "GND" H 7555 5877 50  0000 C CNN
 F 2 "" H 7550 6050 50  0001 C CNN
@@
 $EndComp
 $Comp
-L Device:CP C?
+L Device:CP C2
 U 1 1 607E39E7
 P 4550 5650
-F 0 "C?" H 4432 5604 50  0000 R CNN
+F 0 "C2" H 4432 5604 50  0000 R CNN
 F 1 "100uF" H 4432 5695 50  0000 R CNN
 F 2 "" H 4588 5500 50  0001 C CNN
@@
 	5450 4700 5700 4700
 $Comp
-L power:GND #PWR?
+L power:GND #PWR0107
 U 1 1 607E3A11
 P 4350 4550
-F 0 "#PWR?" H 4350 4300 50  0001 C CNN
+F 0 "#PWR0107" H 4350 4300 50  0001 C CNN
 F 1 "GND" H 4355 4377 50  0000 C CNN
 F 2 "" H 4350 4550 50  0001 C CNN
@@
 Wire Wire Line
 	6200 1550 6200 1450
-Wire Wire Line
-	3300 1700 3400 1700
-Wire Wire Line
-	3400 1700 3400 1850
-Text GLabel 1950 1300 0    50   Input ~ 0
+$Comp
+L power:GND #PWR0110
+U 1 1 60874636
+P 1650 4900
+F 0 "#PWR0110" H 1650 4650 50  0001 C CNN
+F 1 "GND" H 1655 4727 50  0000 C CNN
+F 2 "" H 1650 4900 50  0001 C CNN
+F 3 "" H 1650 4900 50  0001 C CNN
+	1    1650 4900
+	1    0    0    -1
+$EndComp
+Wire Wire Line
+	1650 4450 1650 4900
+$Comp
+L power:+3.3V #PWR0111
+U 1 1 6087C5D7
+P 1750 2350
+F 0 "#PWR0111" H 1750 2200 50  0001 C CNN
+F 1 "+3.3V" H 1765 2523 50  0000 C CNN
+F 2 "" H 1750 2350 50  0001 C CNN
+F 3 "" H 1750 2350 50  0001 C CNN
+	1    1750 2350
+	1    0    0    -1
+$EndComp
+Text GLabel 7800 1800 2    50   Input ~ 0
+10-24VDC-
+Text GLabel 7800 1600 2    50   Input ~ 0
 10-24VDC+
-Text GLabel 3400 1300 2    50   Output ~ 0
+Wire Wire Line
+	4950 1750 4800 1750
+Text GLabel 4950 1750 2    50   Output ~ 0
+3V3DC
+Text GLabel 3950 1750 0    50   Input ~ 0
 15VDC
 Wire Wire Line
-	3300 1300 3400 1300
-Wire Wire Line
-	2100 1300 1950 1300
-Text GLabel 1950 1700 0    50   Input ~ 0
-10-24VDC-
+	4100 1750 3950 1750
+Wire Wire Line
+	4800 1300 4950 1300
+Wire Wire Line
+	4950 1300 4950 1050
+$Comp
+L power:GND #PWR0109
+U 1 1 608533FB
+P 4950 1050
+F 0 "#PWR0109" H 4950 800 50  0001 C CNN
+F 1 "GND" H 4955 877 50  0000 C CNN
+F 2 "" H 4950 1050 50  0001 C CNN
+F 3 "" H 4950 1050 50  0001 C CNN
+	1    4950 1050
+	-1   0    0    1
+$EndComp
+Wire Wire Line
+	3950 1300 3950 1050
+Wire Wire Line
+	4100 1300 3950 1300
+$Comp
+L power:GND #PWR0108
+U 1 1 608492A3
+P 3950 1050
+F 0 "#PWR0108" H 3950 800 50  0001 C CNN
+F 1 "GND" H 3955 877 50  0000 C CNN
+F 2 "" H 3950 1050 50  0001 C CNN
+F 3 "" H 3950 1050 50  0001 C CNN
+	1    3950 1050
+	-1   0    0    1
+$EndComp
+$Comp
+L MP1584EN:MP1584EN U2
+U 1 1 60847279
+P 4450 1550
+F 0 "U2" H 4450 2065 50  0000 C CNN
+F 1 "MP1584EN" H 4450 1974 50  0000 C CNN
+F 2 "" H 4250 1200 50  0001 C CNN
+F 3 "" H 4250 1200 50  0001 C CNN
+	1    4450 1550
+	1    0    0    -1
+$EndComp
+Wire Wire Line
+	2100 1700 1950 1700
 $Comp
 L xl6009:xl6009_buckboost U1
@@
 	1    0    0    -1
 $EndComp
-Wire Wire Line
-	2100 1700 1950 1700
-$Comp
-L MP1584EN:MP1584EN U2
-U 1 1 60847279
-P 4450 1550
-F 0 "U2" H 4450 2065 50  0000 C CNN
-F 1 "MP1584EN" H 4450 1974 50  0000 C CNN
-F 2 "" H 4250 1200 50  0001 C CNN
-F 3 "" H 4250 1200 50  0001 C CNN
-	1    4450 1550
-	1    0    0    -1
-$EndComp
-$Comp
-L power:GND #PWR?
-U 1 1 608492A3
-P 3950 1050
-F 0 "#PWR?" H 3950 800 50  0001 C CNN
-F 1 "GND" H 3955 877 50  0000 C CNN
-F 2 "" H 3950 1050 50  0001 C CNN
-F 3 "" H 3950 1050 50  0001 C CNN
-	1    3950 1050
-	-1   0    0    1
-$EndComp
-Wire Wire Line
-	4100 1300 3950 1300
-Wire Wire Line
-	3950 1300 3950 1050
-$Comp
-L power:GND #PWR?
-U 1 1 608533FB
-P 4950 1050
-F 0 "#PWR?" H 4950 800 50  0001 C CNN
-F 1 "GND" H 4955 877 50  0000 C CNN
-F 2 "" H 4950 1050 50  0001 C CNN
-F 3 "" H 4950 1050 50  0001 C CNN
-	1    4950 1050
-	-1   0    0    1
-$EndComp
-Wire Wire Line
-	4950 1300 4950 1050
-Wire Wire Line
-	4800 1300 4950 1300
-Wire Wire Line
-	4100 1750 3950 1750
-Text GLabel 3950 1750 0    50   Input ~ 0
+Text GLabel 1950 1700 0    50   Input ~ 0
+10-24VDC-
+Wire Wire Line
+	2100 1300 1950 1300
+Wire Wire Line
+	3300 1300 3400 1300
+Text GLabel 3400 1300 2    50   Output ~ 0
 15VDC
-Text GLabel 4950 1750 2    50   Output ~ 0
-3V3DC
-Wire Wire Line
-	4950 1750 4800 1750
+Text GLabel 1950 1300 0    50   Input ~ 0
+10-24VDC+
+Wire Wire Line
+	3400 1700 3400 1850
+Wire Wire Line
+	3300 1700 3400 1700
+$Comp
+L power:GND #PWR07
+U 1 1 60517F01
+P 3400 1850
+F 0 "#PWR07" H 3400 1600 50  0001 C CNN
+F 1 "GND" H 3405 1677 50  0000 C CNN
+F 2 "" H 3400 1850 50  0001 C CNN
+F 3 "" H 3400 1850 50  0001 C CNN
+	1    3400 1850
+	1    0    0    -1
+$EndComp
 $EndSCHEMATC

Commit message: Footprint PCB Time
Parts:
- removed J1: IN1, Connector_PinHeader_2.54mm:PinHeader_1x02_P2.54mm_Vertical, symbol Connector:Conn_01x02_Male
- removed J2: IN2, Connector_PinHeader_2.54mm:PinHeader_1x02_P2.54mm_Vertical, symbol Connector:Conn_01x02_Male
- removed U1: xl6009_buckboost, symbol xl6009:xl6009_buckboost
- removed U2: MP1584EN, symbol MP1584EN:MP1584EN
- added C1, C3: 100uF, Capacitor_THT:CP_Radial_D5.0mm_P2.00mm, symbol Device:CP
- added C2: 0.01uF, Capacitor_THT:C_Disc_D7.5mm_W5.0mm_P5.00mm, symbol Device:C
- added D1: D_Schottky, Diode_THT:D_A-405_P7.62mm_Horizontal, symbol Device:D_Schottky
- added L1: 68uH, Inductor_THT:L_Axial_L14.0mm_D4.5mm_P5.08mm_Vertical_Fastron_LACC, symbol Device:L
- added U1: LM2674M-3.3, Package_DIP:DIP-8_W7.62mm_Socket, symbol Regulator_Switching:LM2674M-3.3
- C4: renamed from C1; footprint (none) -> Capacitor_THT:CP_Radial_D5.0mm_P2.00mm
- C5: renamed from C2; footprint (none) -> Capacitor_THT:CP_Radial_D5.0mm_P2.00mm
- J1: renamed from J3; footprint Connector_BarrelJack:BarrelJack_CUI_PJ-063AH_Horizontal_CircularHoles -> TerminalBlock:TerminalBlock_Altech_AK300-2_P5.00mm
- U3: renamed from U4; footprint (none) -> ZUno:Z-UNO
- renumbered D1 to D2, D2 to D3, R2 to R1, R3 to R2, R4 to R3, R1 to R4, R7 to R6, R8 to R7, R9 to R8, R6 to R9, U3 to U2
Connections:
- net labels removed: 10-24VDC+, 10-24VDC-
- wire segments 84 -> 81
- no-connect marks 0 -> 23

Commit message: Ok cool
Parts:
- J1: footprint TerminalBlock:TerminalBlock_Altech_AK300-2_P5.00mm -> Connector_BarrelJack:BarrelJack_CUI_PJ-063AH_Horizontal_CircularHoles
Changed lines of the file:
@@
 Wire Wire Line
 	5650 1700 5650 1800
-$Comp
-L Connector:Barrel_Jack J1
-U 1 1 6050E38F
-P 7450 1700
-F 0 "J1" H 7507 2025 50  0000 C CNN
-F 1 "Barrel_Jack" H 7507 1934 50  0000 C CNN
-F 2 "TerminalBlock:TerminalBlock_Altech_AK300-2_P5.00mm" H 7500 1660 50  0001 C CNN
-F 3 "~" H 7500 1660 50  0001 C CNN
-	1    7450 1700
-	1    0    0    -1
-$EndComp
 Wire Wire Line
 	7800 1800 7750 1800
@@
 Wire Wire Line
 	4050 1350 4150 1350
+$Comp
+L Connector:Barrel_Jack J1
+U 1 1 6050E38F
+P 7450 1700
+F 0 "J1" H 7507 2025 50  0000 C CNN
+F 1 "Barrel_Jack" H 7507 1934 50  0000 C CNN
+F 2 "Connector_BarrelJack:BarrelJack_CUI_PJ-063AH_Horizontal_CircularHoles" H 7500 1660 50  0001 C CNN
+F 3 "~" H 7500 1660 50  0001 C CNN
+	1    7450 1700
+	1    0    0    -1
+$EndComp
 $EndSCHEMATC
