File: randall-LM358-5-12V-amp.sch (KiCad schematic (older format))
At the start: 28 parts, among them J1 Barrel_Jack, J2 AVR-ISP-6, M1 Fan_3pin, M2 Fan_3pin, Q1 TIP120, Q2 TIP120, U1 LM2674M-3.3, U2 LM358, U3 Z-Uno-Module

Commit message: added drill holes and re-arrange board
Parts:
- U3: symbol ZUno-module:Z-Uno-Module -> randall-LM358-5-12V-amp-rescue:Z-Uno-Module-ZUno-module
Changed lines of the file:
@@
 $EndComp
 $Comp
-L ZUno-module:Z-Uno-Module U3
+L randall-LM358-5-12V-amp-rescue:Z-Uno-Module-ZUno-module U3
 U 1 1 60867D56
 P 2100 3650

Commit message: Ok added an antenna and some keepouts and rerouted a trace or two:
Parts:
- added J3: Antenna Pin, Connector_PinHeader_2.54mm:PinHeader_1x01_P2.54mm_Vertical, symbol Connector:Conn_01x01_Male
Connections:
- net at U3.33 (RF3): now also J3.1 (Pin_1)
- no-connect marks 44 -> 43
Changed lines of the file:
@@
 	0    1    1    0
-$EndComp
-$Comp
-L randall-LM358-5-12V-amp-rescue:Z-Uno-Module-ZUno-module U3
-U 1 1 60867D56
-P 2100 3650
-F 0 "U3" H 2050 4753 60  0000 C CNN
-F 1 "Z-Uno-Module" H 2050 4647 60  0000 C CNN
-F 2 "ZUno Module:Z-UNO Module" H 2100 3650 60  0001 C CNN
-F 3 "" H 2100 3650 60  0001 C CNN
-	1    2100 3650
-	1    0    0    -1
 $EndComp
 Text GLabel 3000 4450 2    50   Input ~ 0
@@
 NoConn ~ 1100 4450
 NoConn ~ 1100 4550
-NoConn ~ 1100 4750
 NoConn ~ 3000 4150
 NoConn ~ 3000 4250
@@
 Text GLabel 2250 6800 3    50   Output ~ 0
 3V3DC
+$Comp
+L Connector:Conn_01x01_Male J3
+U 1 1 6088B474
+P 900 4750
+F 0 "J3" V 962 4794 50  0000 L CNN
+F 1 "Antenna Pin" H 750 4650 50  0000 L CNN
+F 2 "Connector_PinHeader_2.54mm:PinHeader_1x01_P2.54mm_Vertical" H 900 4750 50  0001 C CNN
+F 3 "~" H 900 4750 50  0001 C CNN
+	1    900  4750
+	1    0    0    -1
+$EndComp
+$Comp
+L randall-LM358-5-12V-amp-rescue:Z-Uno-Module-ZUno-module U3
+U 1 1 60867D56
+P 2100 3650
+F 0 "U3" H 2050 4753 60  0000 C CNN
+F 1 "Z-Uno-Module" H 2050 4647 60  0000 C CNN
+F 2 "ZUno Module:Z-UNO Module" H 2100 3650 60  0001 C CNN
+F 3 "" H 2100 3650 60  0001 C CNN
+	1    2100 3650
+	1    0    0    -1
+$EndComp
 $EndSCHEMATC

Commit message: Updating P/N
Parts:
- C1, C3: value 100uF -> 100uF OSCON-SEP
- C4, C5: value 100uF -> 100uF 25v
- D1: value D_Schottky -> 11DQ05TA
- L1: value 68uH -> 68uH B78148E
- M1, M2: value Fan_3pin -> Molex 22282931
- U1: value LM2674M-3.3 -> LM2674N-3.3/NOPB
- U2: value LM358 -> LM358N/NOPB
Other:
- moved on the sheet: C3, L1
Changed lines of the file:
@@
 P 6850 1700
 F 0 "U2" H 6808 1746 50  0000 L CNN
-F 1 "LM358" H 6808 1655 50  0000 L CNN
+F 1 "LM358N/NOPB" H 6808 1655 50  0000 L CNN
 F 2 "Package_DIP:DIP-8_W7.62mm_Socket" H 6850 1700 50  0001 C CNN
 F 3 "http://www.ti.com/lit/ds/symlink/lm2904-n.pdf" H 6850 1700 50  0001 C CNN
@@
 P 7550 3700
 F 0 "M1" H 7708 3696 50  0000 L CNN
-F 1 "Fan_3pin" H 7708 3605 50  0000 L CNN
+F 1 "Molex 22282931" H 7708 3605 50  0000 L CNN
 F 2 "Connector_Molex:Molex_KK-254_AE-6410-03A_1x03_P2.54mm_Vertical" H 7550 3610 50  0001 C CNN
 F 3 "http://www.hardwarecanucks.com/forum/attachments/new-builds/16287d1330775095-help-chassis-power-fan-connectors-motherboard-asus_p8z68.jpg" H 7550 3610 50  0001 C CNN
@@
 P 4550 3600
 F 0 "C4" H 4668 3646 50  0000 L CNN
-F 1 "100uF" H 4668 3555 50  0000 L CNN
+F 1 "100uF 25v" H 4668 3555 50  0000 L CNN
 F 2 "Capacitor_THT:CP_Radial_D5.0mm_P2.00mm" H 4588 3450 50  0001 C CNN
 F 3 "~" H 4550 3600 50  0001 C CNN
@@
 P 5750 3200
 F 0 "U2" H 5700 2850 50  0000 C CNN
-F 1 "LM358" H 5750 2924 50  0000 C CNN
+F 1 "LM358N/NOPB" H 5750 2924 50  0000 C CNN
 F 2 "Package_DIP:DIP-8_W7.62mm_Socket" H 5750 3200 50  0001 C CNN
 F 3 "http://www.ti.com/lit/ds/symlink/lm2904-n.pdf" H 5750 3200 50  0001 C CNN
@@
 P 7550 5750
 F 0 "M2" H 7708 5746 50  0000 L CNN
-F 1 "Fan_3pin" H 7708 5655 50  0000 L CNN
+F 1 "Molex 22282931" H 7708 5655 50  0000 L CNN
 F 2 "Connector_Molex:Molex_KK-254_AE-6410-03A_1x03_P2.54mm_Vertical" H 7550 5660 50  0001 C CNN
 F 3 "http://www.hardwarecanucks.com/forum/attachments/new-builds/16287d1330775095-help-chassis-power-fan-connectors-motherboard-asus_p8z68.jpg" H 7550 5660 50  0001 C CNN
@@
 P 4550 5650
 F 0 "C5" H 4432 5604 50  0000 R CNN
-F 1 "100uF" H 4432 5695 50  0000 R CNN
+F 1 "100uF 25v" H 4432 5695 50  0000 R CNN
 F 2 "Capacitor_THT:CP_Radial_D5.0mm_P2.00mm" H 4588 5500 50  0001 C CNN
 F 3 "~" H 4550 5650 50  0001 C CNN
@@
 P 5750 5250
 F 0 "U2" H 5700 4900 50  0000 C CNN
-F 1 "LM358" H 5750 4974 50  0000 C CNN
+F 1 "LM358N/NOPB" H 5750 4974 50  0000 C CNN
 F 2 "Package_DIP:DIP-8_W7.62mm_Socket" H 5750 5250 50  0001 C CNN
 F 3 "http://www.ti.com/lit/ds/symlink/lm2904-n.pdf" H 5750 5250 50  0001 C CNN
@@
 P 2850 1150
 F 0 "U1" H 2850 1617 50  0000 C CNN
-F 1 "LM2674M-3.3" H 2850 1526 50  0000 C CNN
+F 1 "LM2674N-3.3/NOPB" H 2850 1526 50  0000 C CNN
 F 2 "Package_DIP:DIP-8_W7.62mm_Socket" H 2900 800 50  0001 L CIN
 F 3 "http://www.ti.com/lit/ds/symlink/lm2674.pdf" H 2850 1150 50  0001 C CNN
@@
 P 1850 1100
 F 0 "C1" H 1968 1146 50  0000 L CNN
-F 1 "100uF" H 1968 1055 50  0000 L CNN
+F 1 "100uF OSCON-SEP" H 1600 950 50  0000 L CNN
 F 2 "Capacitor_THT:CP_Radial_D5.0mm_P2.00mm" H 1888 950 50  0001 C CNN
 F 3 "~" H 1850 1100 50  0001 C CNN
@@
 Wire Wire Line
 	3350 1350 3450 1350
-Text GLabel 4150 1650 3    50   Input ~ 0
+Text GLabel 4450 1650 3    50   Input ~ 0
 GND
 Wire Wire Line
@@
 Wire Wire Line
 	2850 1550 2850 1650
-Text GLabel 4400 1350 2    50   Output ~ 0
+Text GLabel 4650 1350 2    50   Output ~ 0
 3V3DC
 $Comp
@@
 P 3450 1500
 F 0 "D1" V 3404 1580 50  0000 L CNN
-F 1 "D_Schottky" V 3495 1580 50  0000 L CNN
+F 1 "11DQ05TA" V 3495 1580 50  0000 L CNN
 F 2 "Diode_THT:D_A-405_P7.62mm_Horizontal" H 3450 1500 50  0001 C CNN
 F 3 "~" H 3450 1500 50  0001 C CNN
@@
 L Device:CP C3
 U 1 1 6087ABE3
-P 4150 1500
-F 0 "C3" H 4268 1546 50  0000 L CNN
-F 1 "100uF" H 4268 1455 50  0000 L CNN
-F 2 "Capacitor_THT:CP_Radial_D5.0mm_P2.00mm" H 4188 1350 50  0001 C CNN
-F 3 "~" H 4150 1500 50  0001 C CNN
-	1    4150 1500
-	1    0    0    -1
-$EndComp
-Wire Wire Line
-	4150 950  4150 1350
-Wire Wire Line
-	3350 950  4150 950
-Connection ~ 4150 1350
-Wire Wire Line
-	4150 1350 4400 1350
+P 4450 1500
+F 0 "C3" H 4568 1546 50  0000 L CNN
+F 1 "100uF OSCON-SEP" H 4200 1400 50  0000 L CNN
+F 2 "Capacitor_THT:CP_Radial_D5.0mm_P2.00mm" H 4488 1350 50  0001 C CNN
+F 3 "~" H 4450 1500 50  0001 C CNN
+	1    4450 1500
+	1    0    0    -1
+$EndComp
+Connection ~ 4450 1350
 $Comp
 L Device:L L1
 U 1 1 60877FA2
-P 3900 1350
-F 0 "L1" V 4090 1350 50  0000 C CNN
-F 1 "68uH" V 3999 1350 50  0000 C CNN
-F 2 "Inductor_THT:L_Axial_L14.0mm_D4.5mm_P5.08mm_Vertical_Fastron_LACC" H 3900 1350 50  0001 C CNN
-F 3 "~" H 3900 1350 50  0001 C CNN
-	1    3900 1350
+P 4050 1350
+F 0 "L1" V 4240 1350 50  0000 C CNN
+F 1 "68uH B78148E" V 4149 1350 50  0000 C CNN
+F 2 "Inductor_THT:L_Axial_L14.0mm_D4.5mm_P5.08mm_Vertical_Fastron_LACC" H 4050 1350 50  0001 C CNN
+F 3 "~" H 4050 1350 50  0001 C CNN
+	1    4050 1350
 	0    -1   -1   0
 $EndComp
 Wire Wire Line
-	3750 1350 3650 1350
-Wire Wire Line
-	4050 1350 4150 1350
+	3900 1350 3650 1350
+Wire Wire Line
+	4200 1350 4450 1350
 $Comp
 L Connector:Barrel_Jack J1
@@
 U 1 1 60867D56
 P 2100 3650
-F 0 "U3" H 2050 4753 60  0000 C CNN
-F 1 "Z-Uno-Module" H 2050 4647 60  0000 C CNN
+F 0 "U3" H 2500 4650 60  0000 C CNN
+F 1 "Z-Uno-Module" H 2550 4500 60  0000 C CNN
 F 2 "ZUno Module:Z-UNO Module" H 2100 3650 60  0001 C CNN
 F 3 "" H 2100 3650 60  0001 C CNN
@@
 	1    0    0    -1
 $EndComp
+Wire Wire Line
+	4450 1350 4650 1350
+Wire Wire Line
+	4450 1350 4450 950
+Wire Wire Line
+	3350 950  4450 950
 $EndSCHEMATC
